Commit message: updated with working sim

File: catkin_ws/install/uuv_descriptions/share/uuv_descriptions/robots/generated/rexrov/robot_description.urdf (robot description, URDF)
Before this commit: robot rexrov, 26 links, 25 joints
Links:
- added link base_link
Joints:
- added joint rexrov/dummy_joint: type fixed, parent base_link, child rexrov/base_link

File: catkin_ws/install/uuv_descriptions/share/uuv_descriptions/urdf/rexrov_base.xacro (robot description, xacro)
@@ -72,4 +72,9 @@
       </collision>
     </link>
+    <link name="base_link"/>
+    <joint name="${namespace}/dummy_joint" type="fixed">
+      <parent link="base_link"/>
+      <child link="${namespace}/base_link"/>
+    </joint>
     <!-- Set up hydrodynamic plugin given as input parameter -->
     <xacro:insert_block name="gazebo"/>
