Commit message: fix: delete build files and make some updates

File: catkin_ws/src/beluga_simulator/robots/beluga_default.xacro (robot description, xacro)
@@ -18,5 +18,5 @@
   <!-- Include the ROV macro file -->
   <xacro:include filename="$(find beluga_simulator)/urdf/beluga_base.xacro"/>
-  <xacro:include filename="$(find beluga_simulator)/urdf/misc.xacro"/>
+  <!-- <xacro:include filename="$(find beluga_simulator)/urdf/misc.xacro"/> -->
   <!-- Create the beluga -->
   <xacro:beluga_base
@@ -25,4 +25,4 @@
     inertial_reference_frame="$(arg inertial_reference_frame)"/>
   <!-- Joint state publisher plugin -->
-  <xacro:default_joint_state_publisher namespace="$(arg namespace)" update_rate="5"/>
+  <!-- <xacro:default_joint_state_publisher namespace="$(arg namespace)" update_rate="5"/> -->
 </robot>

File: catkin_ws/src/beluga_simulator/urdf/beluga_base.xacro (robot description, xacro)
@@ -15,7 +15,7 @@
   <xacro:macro name="beluga_base" params="namespace debug inertial_reference_frame">
   <!-- Import xacros -->
-  <xacro:include filename="$(find beluga_simulator)/models/common.urdf.xacro"/>
-  <xacro:include filename="$(find beluga_simulator)/models/sensor_snippets.xacro"/>
-  <xacro:include filename="$(find beluga_simulator)/models/thruster_snippets.xacro"/>
+  <xacro:include filename="$(find beluga_simulator)/urdf/common.urdf.xacro"/>
+  <xacro:include filename="$(find beluga_simulator)/urdf/sensor_snippets.xacro"/>
+  <xacro:include filename="$(find beluga_simulator)/urdf/thruster_snippets.xacro"/>
   <!-- Define Parameters -->
   <xacro:property name="mass" value="20"/>
@@ -103,44 +103,6 @@
      <child link="${namespace}/base_link"/>
   </joint>
-  <gazebo reference="${namespace}/base_link">
-    <selfCollide>false</selfCollide>
-  </gazebo>
-  <!-- Set up hydrodynamics plugin -->
-  <gazebo>
-    <plugin name="${namespace}_uuv_plugin" filename="libuuv_underwater_object_ros_plugin.so">
-      <fluid_density>${rho}</fluid_density>
-      <flow_velocity_topic>hydrodynamics/current_velocity</flow_velocity_topic>
-      <debug>${debug}</debug>
-      <link name="${namespace}/base_link">
-        <neutrally_bouyant>0</neutrally_bouyant>
-        <volume>${volume}</volume>
-        <box>
-          <width>${y_size}</width>
-          <length>${x_size}</length>
-          <height>${z_size}</height>
-        </box>
-        <center_of_buoyancy>${cob}</center_of_buoyancy>
-          <hydrodynamic_model>
-            <type>fossen</type>
-            <added_mass>
-              3.899   -0.034  -0.517  0.043   -0.828  -0.039
-              -0.034  6.110   0.256   2.047   -0.029  0.314
-              -0.517  0.256   18.300  0.031   -1.932  0.054
-              0.043   2.047   0.031   1.675   -0.050  0.105
-              -0.828  -0.029  -1.932  -0.050  2.213   -0.006
-              -0.039  0.314   0.054   0.105   -0.006  0.622
-            </added_mass>
-            <linear_damping>
-              -9.352  -8.685  -91.050 -10 -10 -5
-            </linear_damping>
-            <quadratic_damping>
-              -93.528 -124.066 -227.626 -20 -20 -15
-            </quadratic_damping>
-          </hydrodynamic_model>
-        </link>
-      </plugin>
-    </gazebo>
-    <xacro:include filename="$(find beluga_simulator)/models/beluga_thrusters.xacro"/>
-    <xacro:include filename="$(find beluga_simulator)/models/beluga_sensors.xacro"/>
+    <xacro:include filename="$(find beluga_simulator)/urdf/beluga_thrusters.xacro"/>
+    <!-- <xacro:include filename="$(find beluga_simulator)/urdf/beluga_sensors.xacro"/> -->
   </xacro:macro>
 </robot>

File: catkin_ws/src/beluga_simulator/urdf/beluga_thrusters.xacro (robot description, xacro)
@@ -14,5 +14,5 @@
 <robot xmlns:xacro="http://www.ros.org/wiki/xacro">
   <!-- Thrusters -->
-  <xacro:include filename="$(find beluga_simulator)/models/beluga_snippets.xacro"/>
+  <xacro:include filename="$(find beluga_simulator)/urdf/beluga_snippets.xacro"/>
   <!-- Left Front Thruster -->
   <xacro:thruster_macro

File: catkin_ws/src/beluga_simulator/urdf/camera_snippets.xacro (robot description, xacro)
@@ -206,21 +206,4 @@
           </noise>
         </camera>
-        <plugin name="camera${suffix}_controller" filename="libuuv_gazebo_ros_camera_plugin.so">
-          <updateRate>${update_rate}</updateRate>
-          <cameraName>${namespace}/camera${suffix}</cameraName>
-          <frameName>${namespace}/camera${suffix}_link</frameName>
-          <attenuationR>0.01</attenuationR>
-          <attenuationG>0.01</attenuationG>
-          <attenuationB>0.003</attenuationB>
-          <backgroundR>0</backgroundR>
-          <backgroundG>0</backgroundG>
-          <backgroundB>0</backgroundB>
-          <!-- required for ros depth cam -->
-          <imageTopicName>${topic}_image</imageTopicName>
-          <pointCloudTopicName>${topic}_cloud</pointCloudTopicName>
-          <depthImageTopicName>${topic}_depth</depthImageTopicName>
-          <depthImageCameraInfoTopicName>${topic}_depth_info</depthImageCameraInfoTopicName>
-          <pointCloudCutoff>10.0</pointCloudCutoff>
-        </plugin>
       </sensor>
     </gazebo>

File: catkin_ws/src/beluga_simulator/urdf/pressure_snippets.xacro (robot description, xacro)
@@ -81,19 +81,4 @@
       <axis xyz="1 0 0"/>
     </joint>
-    <gazebo>
-      <plugin filename="libuuv_gazebo_ros_subsea_pressure_plugin.so" name="libuuv_gazebo_subseapressure${suffix}_plugin">
-        <robot_namespace>${namespace}</robot_namespace> <!-- (string, required): ros namespace in which the messages are published -->
-        <link_name>${namespace}/pressure${suffix}_link</link_name> <!-- (string, required): name of the body which holds the IMU sensor -->
-        <sensor_topic>${topic}</sensor_topic> <!-- (string): name of the sensor output topic and prefix of service names (defaults to imu) -->
-        <update_rate>${update_rate}</update_rate> <!-- Update period of accelerometer and gyroscope [s] -->
-        <saturation>${range}</saturation> <!-- measurement range [kPa] -->
-        <noise_sigma>${noise_sigma}</noise_sigma> <!-- measurement stddev [kPa] -->
-        <noise_amplitude>${noise_amplitude}</noise_amplitude>
-        <estimate_depth_on>${estimateDepth}</estimate_depth_on> <!-- infer depth? -->
-        <standard_pressure>${standardPressure}</standard_pressure> <!-- pressure at sea level (depth 0 m) [kPa] -->
-        <kPa_per_meter>${kPaPerM}</kPa_per_meter> <!-- increase in pressure [kPa] per [m] in increased depth -->
-        <enable_gazebo_messages>false</enable_gazebo_messages>
-      </plugin>
-    </gazebo>
   </xacro:macro>
 </robot>

File: catkin_ws/src/beluga_simulator/urdf/thruster_snippets.xacro (robot description, xacro)
@@ -73,7 +73,5 @@
             thruster_id
             *origin
-            mesh_filename
-            *dynamics
-            *conversion">
+            mesh_filename">
     <joint name="${namespace}/thruster_${thruster_id}_joint" type="continuous">
       <xacro:insert_block name="origin"/>
@@ -107,16 +105,4 @@
       </inertial>
     </link>
-    <gazebo>
-      <plugin name="${namespace}_${thruster_id}_thruster_model" filename="libuuv_thruster_ros_plugin.so">
-        <linkName>${namespace}/thruster_${thruster_id}</linkName>
-        <jointName>${namespace}/thruster_${thruster_id}_joint</jointName>
-        <thrusterID>${thruster_id}</thrusterID>
-        <xacro:insert_block name="dynamics"/>
-        <xacro:insert_block name="conversion"/>
-      </plugin>
-    </gazebo>
-    <gazebo reference="${namespace}/thruster_${thruster_id}">
-      <selfCollide>false</selfCollide>
-    </gazebo>
   </xacro:macro>
   <!--
@@ -137,6 +123,4 @@
       mesh_filename="${mesh_filename}">
       <xacro:insert_block name="origin"/>
-      <xacro:rotor_dyn_first_order_macro time_constant="${dyn_time_constant}"/>
-      <xacro:thruster_cf_basic_macro rotor_constant="${rotor_constant}"/>
     </xacro:generic_thruster_macro>
   </xacro:macro>
